Commit message: Right hand closes into a fist (D20); balance: MuJoCo --push test and ramped-push training run (D19)
- build_g1_pingpang_models.py generates meshes/right_fist.STL and uses it as the right_rubber_hand
  visual (URDF + MJCF); racket pose, mass, inertia, collisions unchanged.
- mujoco_eval_onnx.py --push V_XY W_RPY / --push-window-s: one random base-velocity shove per ball
  (own RNG stream).
- mdp.push_by_setting_velocity_ramped + train.py domain_rand.push_* knobs install events.push_robot.
- HOPEPingPongUnitreeG1_FH_XC_RALLY_BAL: rally recipe + shoves ramped to +-0.5 m/s over 3000 iters.

Co-Authored-By: Claude Opus 5.5 <noreply@anthropic.com>

File: unitree/URDF/g1_29dof_pingpang/urdf/g1_29dof_pingpang.urdf (robot description, URDF)
Before this commit: robot g1_29dof_pingpang, 42 links, 41 joints
Links:
- link right_rubber_hand: geometry visual mesh filename=../meshes/right_fist.STL

Commit message: Fist grip (D20, revised): racket perpendicular to the forearm on a separate G1 model; forearm model back to the open hand
- build_g1_pingpang_models.py: Mount variants FOREARM (unchanged, every existing run) and FIST
  (handle across the closed fist, blade origin (0.083, 0.0226, 0.14), rpy (0, -pi/2, 0), red face = palm)
  -> unitree/URDF/g1_29dof_pingpang_fist/ with a generated fist mesh.
- robots/g1.py G1_FIST_MOUNT_* + G1_RACKET_MOUNTS; train.py task key g1_racket_mount: fist swaps the
  Isaac asset (own prepared dir assets/unitree_g1_fist) and the racket-target mount.
- retarget_a3_clip_to_g1_ik.py --mount fist -> g1ikfist_hope_{forehand,backhand} clips.
- Task HOPEPingPongUnitreeG1_FH_FIST (rally + shoves + fist mount + fist IK clips).
- g1_smoke.sbatch gets the AVOID_GPU_IDX guard.

Co-Authored-By: Claude Opus 5.5 <noreply@anthropic.com>

File: unitree/URDF/g1_29dof_pingpang/urdf/g1_29dof_pingpang.urdf (robot description, URDF)
Before this commit: robot g1_29dof_pingpang, 42 links, 41 joints
Links:
- link right_rubber_hand: geometry visual mesh filename=../../g1_description/meshes/right_rubber_hand.STL
